File: PCB/SensLord/SensLord.kicad_pcb (KiCad board)
At the start: 2 copper layers, 187.5 x 45 mm, 26 parts, among them J111 USB_B_Micro, Q120 IRLML6402, U1 ESP32-C6-MINI-1, U110 MCP73831-2-OT, U140 MCP1700x-330xxTT

Commit message: testing circuit ..
Parts:
- moved TP5 16.2 mm to (93.8, 42.2)
- moved R131 11.3 mm to (67.8, 46.2)
- moved R132 11.3 mm to (71.9, 46.2)
- moved TP4 10.4 mm to (90.8, 42.2)
- moved U140 10.1 mm to (95.3, 34.8)
- moved C123 10.1 mm to (88.3, 33.7)
- moved C124 10.1 mm to (91.3, 33.7)
- moved Q120 10.1 mm to (93.3, 38.2)
- moved R121 10.1 mm to (88.3, 38.6)
- moved R122 10.1 mm to (90.3, 38.6)
- moved BT130 8.02 mm to (63.2, 49.7)
- moved D141 6.10 mm to (99.5, 32.5), turned to 180 degrees
- moved TP3 4.42 mm to (87.5, 42.2)
- moved JP112 2.62 mm to (77.0, 41.5)
- moved TP2 1.75 mm to (84.5, 42.2)
Changed lines of the file:
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@@
 	(footprint "Package_TO_SOT_SMD:SOT-23"
 		(layer "F.Cu")
-		(at 95.9375 47.95)
+		(at 93.2875 38.2)
 		(descr "SOT, 3 Pin (JEDEC TO-236 Var AB https://www.jedec.org/document_search?search_api_views_fulltext=TO-236), generated with kicad-footprint-generator ipc_gullwing_generator.py")
 		(tags "SOT TO_SOT_SMD")
@@
 	(footprint "TestPoint:TestPoint_Pad_D1.0mm"
 		(layer "F.Cu")
-		(at 84.5 55.5)
+		(at 93.75 42.25)
 		(descr "SMD pad as test Point, diameter 1.0mm")
 		(tags "test point SMD pad")
@@
 	(footprint "Resistor_SMD:R_0603_1608Metric"
 		(layer "F.Cu")
-		(at 93 48.325 -90)
+		(at 90.35 38.575 -90)
 		(descr "Resistor SMD 0603 (1608 Metric), square (rectangular) end terminal, IPC-7351 nominal, (Body size source: IPC-SM-782 page 72, https://www.pcb-3d.com/wordpress/wp-content/uploads/ipc-sm-782a_amendment_1_and_2.pdf), generated with kicad-footprint-generator")
 		(tags "resistor")
@@
 	(footprint "TestPoint:TestPoint_Pad_D1.0mm"
 		(layer "F.Cu")
-		(at 84.5 40.5)
+		(at 84.5 42.25)
 		(descr "SMD pad as test Point, diameter 1.0mm")
 		(tags "test point SMD pad")
@@
 	(footprint "Package_TO_SOT_SMD:SOT-23"
 		(layer "F.Cu")
-		(at 98 44.5625 -90)
+		(at 95.3 34.8125 -90)
 		(descr "SOT, 3 Pin (JEDEC TO-236 Var AB https://www.jedec.org/document_search?search_api_views_fulltext=TO-236), generated with kicad-footprint-generator ipc_gullwing_generator.py")
 		(tags "SOT TO_SOT_SMD")
@@
 		(tags "capacitor")
 		(property "Reference" "C117"
-			(at 4.975 0 90)
+			(at -0.025 1.75 90)
 			(layer "F.SilkS")
 			(effects
@@
 		)
 		(property "Value" "4.7uF"
-			(at 9.975 0 90)
+			(at -0.025 0 90)
 			(layer "F.Fab")
 			(effects
@@
 	(footprint "Resistor_SMD:R_0603_1608Metric"
 		(layer "F.Cu")
-		(at 91 48.325 90)
+		(at 88.35 38.575 90)
 		(descr "Resistor SMD 0603 (1608 Metric), square (rectangular) end terminal, IPC-7351 nominal, (Body size source: IPC-SM-782 page 72, https://www.pcb-3d.com/wordpress/wp-content/uploads/ipc-sm-782a_amendment_1_and_2.pdf), generated with kicad-footprint-generator")
 		(tags "resistor")
@@
 	(footprint "Capacitor_SMD:C_1206_3216Metric"
 		(layer "F.Cu")
-		(at 91 43.475 -90)
+		(at 88.35 33.725 -90)
 		(descr "Capacitor SMD 1206 (3216 Metric), square (rectangular) end terminal, IPC-7351 nominal, (Body size source: IPC-SM-782 page 76, https://www.pcb-3d.com/wordpress/wp-content/uploads/ipc-sm-782a_amendment_1_and_2.pdf), generated with kicad-footprint-generator")
 		(tags "capacitor")
@@
 		)
 		(property "Value" "4.7uF"
-			(at -9.475 0 90)
+			(at 0.025 0 90)
 			(layer "F.Fab")
 			(effects
@@
 	(footprint "Resistor_SMD:R_0603_1608Metric"
 		(layer "F.Cu")
-		(at 69 57.5)
+		(at 67.775 46.25)
 		(descr "Resistor SMD 0603 (1608 Metric), square (rectangular) end terminal, IPC-7351 nominal, (Body size source: IPC-SM-782 page 72, https://www.pcb-3d.com/wordpress/wp-content/uploads/ipc-sm-782a_amendment_1_and_2.pdf), generated with kicad-footprint-generator")
 		(tags "resistor")
@@
 	(footprint "Diode_SMD:D_SOD-323F"
 		(layer "F.Cu")
-		(at 98.4 38.5)
+		(at 99.5 32.5 180)
 		(descr "SOD-323F http://www.nxp.com/documents/outline_drawing/SOD323F.pdf")
 		(tags "SOD-323F")
@@
 		)
 		(property "Value" "BAT54J"
-			(at 0.1 1.9 0)
+			(at 0 0 0)
 			(layer "F.Fab")
 			(effects
@@
 		)
 		(property "Datasheet" "https://assets.nexperia.com/documents/data-sheet/BAT54J.pdf"
-			(at 0 0 0)
+			(at 0 0 180)
 			(unlocked yes)
 			(layer "F.Fab")
@@
 		)
 		(property "Description" "30V 200mA Schottky diode, SOD-323F"
-			(at 0 0 0)
+			(at 0 0 180)
 			(unlocked yes)
 			(layer "F.Fab")
@@
 		(attr smd)
 		(fp_line
-			(start -1.61 -0.85)
-			(end -1.61 0.85)
+			(start -1.61 0.85)
+			(end 1.05 0.85)
 			(stroke
 				(width 0.12)
@@
 		)
 		(fp_line
-			(start -1.61 0.85)
-			(end 1.05 0.85)
+			(start -1.61 -0.85)
+			(end -1.61 0.85)
 			(stroke
 				(width 0.12)
@@
 		)
 		(fp_line
-			(start -1.6 -0.95)
-			(end -1.6 0.95)
+			(start 1.6 -0.95)
+			(end 1.6 0.95)
 			(stroke
 				(width 0.05)
@@
 		)
 		(fp_line
-			(start -1.6 -0.95)
-			(end 1.6 -0.95)
+			(start -1.6 0.95)
+			(end 1.6 0.95)
 			(stroke
 				(width 0.05)
@@
 		)
 		(fp_line
-			(start -1.6 0.95)
-			(end 1.6 0.95)
+			(start -1.6 -0.95)
+			(end 1.6 -0.95)
 			(stroke
 				(width 0.05)
@@
 		)
 		(fp_line
-			(start 1.6 -0.95)
-			(end 1.6 0.95)
+			(start -1.6 -0.95)
+			(end -1.6 0.95)
 			(stroke
 				(width 0.05)
@@
 		)
 		(fp_line
-			(start -0.9 -0.7)
-			(end 0.9 -0.7)
+			(start 0.9 0.7)
+			(end -0.9 0.7)
 			(stroke
 				(width 0.1)
@@
 		)
 		(fp_line
-			(start -0.9 0.7)
-			(end -0.9 -0.7)
+			(start 0.9 -0.7)
+			(end 0.9 0.7)
 			(stroke
 				(width 0.1)
@@
 		)
 		(fp_line
-			(start -0.3 -0.35)
-			(end -0.3 0.35)
+			(start 0.2 0.35)
+			(end -0.3 0)
 			(stroke
 				(width 0.1)
@@
 		)
 		(fp_line
-			(start -0.3 0)
-			(end -0.5 0)
+			(start 0.2 0)
+			(end 0.45 0)
 			(stroke
 				(width 0.1)
@@
 		)
 		(fp_line
-			(start -0.3 0)
-			(end 0.2 -0.35)
+			(start 0.2 -0.35)
+			(end 0.2 0.35)
 			(stroke
 				(width 0.1)
@@
 		)
 		(fp_line
-			(start 0.2 -0.35)
-			(end 0.2 0.35)
+			(start -0.3 0)
+			(end 0.2 -0.35)
 			(stroke
 				(width 0.1)
@@
 		)
 		(fp_line
-			(start 0.2 0)
-			(end 0.45 0)
+			(start -0.3 0)
+			(end -0.5 0)
 			(stroke
 				(width 0.1)
@@
 		)
 		(fp_line
-			(start 0.2 0.35)
-			(end -0.3 0)
+			(start -0.3 -0.35)
+			(end -0.3 0.35)
 			(stroke
 				(width 0.1)
@@
 		)
 		(fp_line
-			(start 0.9 -0.7)
-			(end 0.9 0.7)
+			(start -0.9 0.7)
+			(end -0.9 -0.7)
 			(stroke
 				(width 0.1)
@@
 		)
 		(fp_line
-			(start 0.9 0.7)
-			(end -0.9 0.7)
+			(start -0.9 -0.7)
+			(end 0.9 -0.7)
 			(stroke
 				(width 0.1)
@@
 		)
 		(pad "1" smd roundrect
-			(at -1.1 0)
+			(at -1.1 0 180)
 			(size 0.5 0.5)
 			(layers "F.Cu" "F.Mask" "F.Paste")
@@
 		)
 		(pad "2" smd roundrect
-			(at 1.1 0)
+			(at 1.1 0 180)
 			(size 0.5 0.5)
 			(layers "F.Cu" "F.Mask" "F.Paste")
@@
 		(tags "capacitor")
 		(property "Reference" "C115"
-			(at 4.975 0 90)
+			(at -0.025 -1.75 90)
 			(layer "F.SilkS")
 			(effects
@@
 		)
 		(property "Value" "4.7uF"
-			(at 9.975 0 90)
+			(at -0.025 0 90)
 			(layer "F.Fab")
 			(effects
@@
 	(footprint "Resistor_SMD:R_0603_1608Metric"
 		(layer "F.Cu")
-		(at 73.15 57.5)
+		(at 71.925 46.25)
 		(descr "Resistor SMD 0603 (1608 Metric), square (rectangular) end terminal, IPC-7351 nominal, (Body size source: IPC-SM-782 page 72, https://www.pcb-3d.com/wordpress/wp-content/uploads/ipc-sm-782a_amendment_1_and_2.pdf), generated with kicad-footprint-generator")
 		(tags "resistor")
@@
 	(footprint "Connector_PinHeader_2.54mm:PinHeader_2x02_P2.54mm_Vertical_SMD"
 		(layer "F.Cu")
-		(at 76.23 44.025 -90)
+		(at 77.02 41.525 -90)
 		(descr "surface-mounted straight pin header, 2x02, 2.54mm pitch, double rows")
 		(tags "Surface mounted pin header SMD 2x02 2.54mm double row")
@@
 	(footprint "Capacitor_SMD:C_1206_3216Metric"
 		(layer "F.Cu")
-		(at 94 43.475 90)
+		(at 91.35 33.725 90)
 		(descr "Capacitor SMD 1206 (3216 Metric), square (rectangular) end terminal, IPC-7351 nominal, (Body size source: IPC-SM-782 page 76, https://www.pcb-3d.com/wordpress/wp-content/uploads/ipc-sm-782a_amendment_1_and_2.pdf), generated with kicad-footprint-generator")
 		(tags "capacitor")
@@
 		)
 		(property "Value" "4.7uF"
-			(at 9.475 0 90)
+			(at -0.025 0.15 90)
 			(layer "F.Fab")
 			(effects
@@
 	(footprint "TestPoint:TestPoint_Pad_D1.0mm"
 		(layer "F.Cu")
-		(at 84.5 45.5)
+		(at 87.5 42.25)
 		(descr "SMD pad as test Point, diameter 1.0mm")
 		(tags "test point SMD pad")
@@
 	(footprint "Connector_PinHeader_2.54mm:PinHeader_1x02_P2.54mm_Vertical"
 		(layer "F.Cu")
-		(at 63.825 57.725)
+		(at 63.25 49.725)
 		(descr "Through hole straight pin header, 1x02, 2.54mm pitch, single row")
 		(tags "Through hole pin header THT 1x02 2.54mm single row")
@@
 	(footprint "TestPoint:TestPoint_Pad_D1.0mm"
 		(layer "F.Cu")
-		(at 84.5 50.5)
+		(at 90.75 42.25)
 		(descr "SMD pad as test Point, diameter 1.0mm")
 		(tags "test point SMD pad")
@@
 	)
 	(via
-		(at 73.975 57.5)
+		(at 72.75 46.25)
 		(size 0.6)
 		(drill 0.3)
@@
 	)
 	(via
-		(at 98.95 43.625)
+		(at 96.25 33.875)
 		(size 0.6)
 		(drill 0.3)
@@
 	)
 	(via
-		(at 94 42)
+		(at 91.35 32.25)
 		(size 0.6)
 		(drill 0.3)
